File: hardware/board.kicad_sch (KiCad schematic)
At the start: 13 parts, among them J1 Power In, J2 LED Strip, Q1 IRF540N, Q2 IRF540N, Q3 IRF540N, SW1 Door Switch 1, SW2 Door Switch 2, U1 L7805, U2 ESP32-DevKitC

Commit message: Swapped IRF540Ns for TIP41Cs for weird red LED behaviour reasons.
Parts:
- removed Q1, Q2, Q3: IRF540N, Package_TO_SOT_THT:TO-220-3_Vertical, symbol Transistor_FET:IRF540N
- added Q1, Q2, Q3: TIP41C, Package_TO_SOT_THT:TO-220-3_Vertical, symbol Transistor_BJT:TIP41C
Connections:
- net BlueOut: now also Q3.2 (C)
- net GND: now also Q1.3 (E), Q2.3 (E), Q3.3 (E)
- net GreenOut: now also Q2.2 (C)
- net RedOut: now also Q1.2 (C)
- net at U2.25 (GPIO0/BOOT/ADC2_CH1): now also Q2.1 (B)
- net at U2.24 (ADC2_CH2/GPIO2): now also Q1.1 (B)
- net at U2.26 (ADC2_CH0/GPIO4): now also Q3.1 (B)

Commit message: Changed LED strip output pins to fix possible issue with bootstrapping on IO0 which I totally should have seen coming.
Connections:
- net at Q3.1 (B): now also U2.11 (ADC2_CH7/GPIO27); no longer U2.26 (ADC2_CH0/GPIO4)
- net at U2.10 (DAC_2/ADC2_CH9/GPIO26): now also Q2.1 (B)
- net at U2.24 (ADC2_CH2/GPIO2): no longer Q1.1 (B)
- net at U2.25 (GPIO0/BOOT/ADC2_CH1): no longer Q2.1 (B)
- net at U2.9 (DAC_1/ADC2_CH8/GPIO25): now also Q1.1 (B)
Changed lines of the file:
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@@
-	(wire
-		(pts
-			(xy 209.55 91.44) (xy 209.55 130.81)
-		)
-		(stroke
-			(width 0)
-			(type default)
-		)
-	)
 	(wire
 		(pts
@@
 	(wire
 		(pts
-			(xy 213.36 88.9) (xy 213.36 74.93)
-		)
-		(stroke
-			(width 0)
-			(type default)
-		)
-	)
-	(wire
-		(pts
-			(xy 194.31 91.44) (xy 209.55 91.44)
-		)
-		(stroke
-			(width 0)
-			(type default)
-		)
-	)
-	(wire
-		(pts
 			(xy 209.55 156.21) (xy 207.01 156.21)
 		)
@@
 	(wire
 		(pts
-			(xy 194.31 88.9) (xy 213.36 88.9)
-		)
-		(stroke
-			(width 0)
-			(type default)
-		)
-	)
-	(wire
-		(pts
 			(xy 260.35 92.71) (xy 257.81 92.71)
 		)
@@
 	(wire
 		(pts
+			(xy 194.31 111.76) (xy 210.82 111.76)
+		)
+		(stroke
+			(width 0)
+			(type default)
+		)
+	)
+	(wire
+		(pts
 			(xy 105.41 81.28) (xy 95.25 81.28)
 		)
@@
 	(wire
 		(pts
+			(xy 194.31 109.22) (xy 209.55 109.22)
+		)
+		(stroke
+			(width 0)
+			(type default)
+		)
+	)
+	(wire
+		(pts
 			(xy 86.36 88.9) (xy 86.36 91.44)
 		)
@@
 	(wire
 		(pts
-			(xy 213.36 74.93) (xy 223.52 74.93)
-		)
-		(stroke
-			(width 0)
-			(type default)
-		)
-	)
-	(wire
-		(pts
 			(xy 93.98 81.28) (xy 95.25 81.28)
 		)
@@
 	(wire
 		(pts
+			(xy 194.31 114.3) (xy 213.36 114.3)
+		)
+		(stroke
+			(width 0)
+			(type default)
+		)
+	)
+	(wire
+		(pts
 			(xy 45.72 81.28) (xy 46.99 81.28)
 		)
@@
 	(wire
 		(pts
-			(xy 194.31 86.36) (xy 210.82 86.36)
-		)
-		(stroke
-			(width 0)
-			(type default)
-		)
-	)
-	(wire
-		(pts
 			(xy 105.41 69.85) (xy 105.41 81.28)
 		)
@@
 	(wire
 		(pts
+			(xy 210.82 111.76) (xy 210.82 102.87)
+		)
+		(stroke
+			(width 0)
+			(type default)
+		)
+	)
+	(wire
+		(pts
+			(xy 209.55 74.93) (xy 223.52 74.93)
+		)
+		(stroke
+			(width 0)
+			(type default)
+		)
+	)
+	(wire
+		(pts
 			(xy 72.39 57.15) (xy 259.08 57.15)
 		)
@@
 	(wire
 		(pts
+			(xy 213.36 130.81) (xy 223.52 130.81)
+		)
+		(stroke
+			(width 0)
+			(type default)
+		)
+	)
+	(wire
+		(pts
+			(xy 209.55 109.22) (xy 209.55 74.93)
+		)
+		(stroke
+			(width 0)
+			(type default)
+		)
+	)
+	(wire
+		(pts
 			(xy 105.41 87.63) (xy 105.41 91.44)
 		)
@@
 	(wire
 		(pts
+			(xy 213.36 114.3) (xy 213.36 130.81)
+		)
+		(stroke
+			(width 0)
+			(type default)
+		)
+	)
+	(wire
+		(pts
 			(xy 210.82 102.87) (xy 223.52 102.87)
 		)
@@
 	(wire
 		(pts
-			(xy 209.55 130.81) (xy 223.52 130.81)
-		)
-		(stroke
-			(width 0)
-			(type default)
-		)
-	)
-	(wire
-		(pts
 			(xy 260.35 95.25) (xy 257.81 95.25)
 		)
@@
 		)
 		(stroke
-			(width 0)
-			(type default)
-		)
-	)
-	(wire
-		(pts
-			(xy 210.82 86.36) (xy 210.82 102.87)
-		)
-		(stroke

Commit message: #3: Finally gave the schematic an MO number like my other projects!
Other:
- title: (none) -> MO-014 Quick-and-Dirty Lights
Changed lines of the file:
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@@
 	(generator_version "10.0")
 	(paper "A4")
+	(title_block
+		(title "MO-014 Quick-and-Dirty Lights")
+		(date "2026-08-08")
+		(rev "v1.0")
+	)
 	(text "Quick-and-Dirty Lights"
 		(exclude_from_sim no)

Commit message: Trivial change to correct reference schematic.
Connections:
- net at SW1.1: now also U2.24 (ADC2_CH2/GPIO2); no longer U2.30 (GPIO18)
- net at U2.26 (ADC2_CH0/GPIO4): now also SW2.1
- net at U2.31 (GPIO19): no longer SW2.1
Changed lines of the file:
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@@
 	(wire
 		(pts
-			(xy 204.47 99.06) (xy 204.47 146.05)
+			(xy 204.47 91.44) (xy 204.47 146.05)
+		)
+		(stroke
+			(width 0)
+			(type default)
+		)
+	)
+	(wire
+		(pts
+			(xy 207.01 88.9) (xy 194.31 88.9)
 		)
 		(stroke
@@
 	(wire
 		(pts
+			(xy 207.01 88.9) (xy 207.01 156.21)
+		)
+		(stroke
+			(width 0)
+			(type default)
+		)
+	)
+	(wire
+		(pts
+			(xy 204.47 91.44) (xy 194.31 91.44)
+		)
+		(stroke
+			(width 0)
+			(type default)
+		)
+	)
+	(wire
+		(pts
 			(xy 209.55 156.21) (xy 207.01 156.21)
 		)
@@
 	(wire
 		(pts
-			(xy 194.31 99.06) (xy 204.47 99.06)
-		)
-		(stroke
-			(width 0)
-			(type default)
-		)
-	)
-	(wire
-		(pts
 			(xy 231.14 156.21) (xy 234.95 156.21)
 		)
@@
 	(wire
 		(pts
-			(xy 207.01 156.21) (xy 207.01 96.52)
-		)
-		(stroke
-			(width 0)
-			(type default)
-		)
-	)
-	(wire
-		(pts
 			(xy 213.36 130.81) (xy 223.52 130.81)
 		)
@@
 		)
 		(stroke
-			(width 0)
-			(type default)
-		)
-	)
-	(wire
-		(pts
-			(xy 207.01 96.52) (xy 194.31 96.52)
-		)
-		(stroke
